Commit message: Displaying TF works properly

File: models/eugen/xacro/simple_ackermann.xacro (robot description, xacro)
@@ -1,4 +1,4 @@
 <?xml version="1.0"?>
-<robot xmlns:xacro="http://www.ros.org/wiki/xacro" name="simple_ackermann" >
+<robot xmlns:xacro="http://ros.org/wiki/xacro" name="simple_ackermann" >
 	<xacro:include filename="$(find realsense_gazebo_plugin)/models/eugen/xacro/simple_ackermann_rear_wheel.xacro"/>
 	<xacro:include filename="$(find realsense_gazebo_plugin)/models/eugen/xacro/simple_ackermann_front_wheel.xacro"/>

File: models/eugen/xacro/simple_ackermann_front_wheel.xacro (robot description, xacro)
@@ -1,4 +1,4 @@
 <?xml version="1.0"?>
-<robot xmlns:xacro="http://www.ros.org/wiki/xacro">
+<robot xmlns:xacro="http://ros.org/wiki/xacro">
 	<!--<xacro:property name="pi" value="3.1415926535897931" />-->
 	<xacro:macro name="default_inertial" params="mass">

File: models/eugen/xacro/simple_ackermann_rear_wheel.xacro (robot description, xacro)
@@ -1,4 +1,4 @@
 <?xml version="1.0"?>
-<robot xmlns:xacro="http://www.ros.org/wiki/xacro" name="simple_ackermann" >
+<robot xmlns:xacro="http://ros.org/wiki/xacro" name="simple_ackermann" >
 	<xacro:macro name="default_inertial" params="mass">
 		<inertial>

File: models/realsense_camera_ros/child_model.urdf.xacro (robot description, xacro)
@@ -3,9 +3,12 @@
   <!--<plugin name="realsense_plugin" filename="librealsense_gazebo_plugin.so"/> -->
   <!--<static>false</static> -->
-		<joint name="base_link_to_camera_link" type="fixed">
-			<origin xyz="-0.1 0.0 5.1" rpy="0.0 0.0 0.0"/>
-			<parent link="base_link"/>
-			<child link="camera_link"/>
-		</joint>
+	<xacro:property name="camera_base_x_" value="0.0" />
+	<xacro:property name="camera_base_y_" value="0.0" />
+	<xacro:property name="camera_base_z_" value="0.2" />
+  <joint name="base_link_to_camera_link" type="fixed">
+    <origin xyz="${camera_base_x_} ${camera_base_y_} ${camera_base_z_}" rpy="0.0 0.0 0.0"/>
+    <parent link="base_link"/>
+    <child link="camera_link"/>
+  </joint>
   <link name="camera_link">
     <pose>0 0 0.015 0 0 0</pose>
@@ -26,5 +29,9 @@
   </link>
   <gazebo>
-    <plugin name="realsense_plugin" filename="librealsense_gazebo_plugin.so"/>
+    <plugin name="realsense_plugin" filename="librealsense_gazebo_plugin.so">
+      <camera_base_x>${camera_base_x_}</camera_base_x>
+      <camera_base_y>${camera_base_y_}</camera_base_y>
+      <camera_base_z>${camera_base_z_}</camera_base_z>
+    </plugin>
   </gazebo>
   <gazebo reference="camera_link">
@@ -34,5 +41,5 @@
         <update_rate>60</update_rate>
         <visualize>1</visualize>
-        <camera name="__default__">
+        <camera name="rgb_camera">
           <horizontal_fov>1.047</horizontal_fov>
           <image>
@@ -57,5 +64,5 @@
         <update_rate>60</update_rate>
         <visualize>0</visualize>
-        <camera name="__default__">
+        <camera name="ir_1_camera">
           <horizontal_fov>1.047</horizontal_fov>
           <image>
@@ -80,5 +87,5 @@
         <update_rate>60</update_rate>
         <visualize>0</visualize>
-        <camera name="__default__">
+        <camera name="ir_2_camera">
           <horizontal_fov>1.047</horizontal_fov>
           <image>
@@ -103,5 +110,5 @@
         <update_rate>60</update_rate>
         <visualize>0</visualize>
-        <camera name="__default__">
+        <camera name="depth_camera">
           <horizontal_fov>1.047</horizontal_fov>
           <image>

Commit message: updated realsense xacro

File: models/eugen/xacro/simple_ackermann.xacro (robot description, xacro)
@@ -1,9 +1,4 @@
 <?xml version="1.0"?>
 <robot xmlns:xacro="http://ros.org/wiki/xacro" name="simple_ackermann" >
-	<xacro:include filename="$(find realsense_gazebo_plugin)/models/eugen/xacro/simple_ackermann_rear_wheel.xacro"/>
-	<xacro:include filename="$(find realsense_gazebo_plugin)/models/eugen/xacro/simple_ackermann_front_wheel.xacro"/>
-	<xacro:include filename="$(find realsense_gazebo_plugin)/models/eugen/xacro/simple_ackermann_plugin.xacro"/>
-	<!--xacro:include filename="$(find realsense_gazebo_plugin)/models/eugen/xacro/simple_drive.xacro"/>-->
-	<xacro:include filename="$(find realsense_gazebo_plugin)/models/realsense_camera_ros/child_model.urdf.xacro"/>
 	<xacro:property name="height" value="0.01" />
 	<xacro:property name="wheelbase" value="0.26" />
@@ -12,4 +7,11 @@
 	<!--xacro:property name="wheelwidth" value="0.001" /-->
 	<xacro:property name="wheelwidth" value="0.0275" />
+	<xacro:property name="ackermann_x_offset" value="-0.09" />
+	<xacro:property name="ackermann_z_offset" value="-0.03" />
+	<xacro:include filename="$(find realsense_gazebo_plugin)/models/eugen/xacro/simple_ackermann_rear_wheel.xacro"/>
+	<xacro:include filename="$(find realsense_gazebo_plugin)/models/eugen/xacro/simple_ackermann_front_wheel.xacro"/>
+	<xacro:include filename="$(find realsense_gazebo_plugin)/models/eugen/xacro/simple_ackermann_plugin.xacro"/>
+	<!--xacro:include filename="$(find realsense_gazebo_plugin)/models/eugen/xacro/simple_drive.xacro"/>-->
+	<xacro:include filename="$(find realsense_gazebo_plugin)/models/realsense_camera_ros/realsense.xacro"/>
 	<xacro:macro name="box_inertial" params="x y z mass">
 		<inertial>

File: models/eugen/xacro/simple_ackermann_plugin.xacro (robot description, xacro)
@@ -13,5 +13,5 @@
 					<robotBaseFrame>base_link</robotBaseFrame>
 					<GazeboDebug>false</GazeboDebug>
-					<Wheelbase>0.26</Wheelbase>
+					<Wheelbase>${wheelbase}</Wheelbase>
 					<Track>0.1525</Track>
 					<SteeringWidth>0.095</SteeringWidth>
@@ -38,4 +38,5 @@
                     <bodyName>base_link</bodyName>
                     <topicName>odom_gt</topicName>
+                    <xyzOffset>${ackermann_x_offset} 0 ${ackermann_z_offset}</xyzOffset>
                     <updateRate>30.0</updateRate>
                 </plugin>

File: models/realsense_camera_ros/realsense.xacro (robot description, xacro)
@@ -33,4 +33,6 @@
       <camera_base_y>${camera_base_y_}</camera_base_y>
       <camera_base_z>${camera_base_z_}</camera_base_z>
+      <ackermann_x_offset_plugin>${ackermann_x_offset}</ackermann_x_offset_plugin>
+      <ackermann_z_offset_plugin>${ackermann_z_offset}</ackermann_z_offset_plugin>
       <robotNamespace>ackermann</robotNamespace>
       <FixedFrame>map</FixedFrame>

Commit message: update

File: models/eugen/xacro/simple_ackermann.xacro (robot description, xacro)
@@ -7,5 +7,5 @@
 	<!--xacro:property name="wheelwidth" value="0.001" /-->
 	<xacro:property name="wheelwidth" value="0.0275" />
-	<xacro:property name="ackermann_x_offset" value="-0.09" />
+	<xacro:property name="ackermann_x_offset" value="-0.095" />
 	<xacro:property name="ackermann_z_offset" value="-0.03" />
 	<xacro:include filename="$(find realsense_gazebo_plugin)/models/eugen/xacro/simple_ackermann_rear_wheel.xacro"/>
